File: pcie-mini-breakout.sch (KiCad schematic (older format))
At the start: 3 parts, among them J1 PCIe Mini, J2 Breakout, J3 MIPI Camera

Commit message: fix connector symbol errors in schematics
Parts:
- J1: symbol Conn_02x26_Odd_Even -> Connector_Generic:Conn_02x26_Odd_Even
- J2: symbol Conn_02x26_Counter_Clockwise -> Connector_Generic:Conn_02x26_Counter_Clockwise
- J3: symbol Conn_01x15 -> Connector_Generic:Conn_01x15
Changed lines of the file:
@@
-EESchema Schematic File Version 2
-LIBS:power
-LIBS:device
-LIBS:switches
-LIBS:relays
-LIBS:motors
-LIBS:transistors
-LIBS:conn
-LIBS:linear
-LIBS:regul
-LIBS:74xx
-LIBS:cmos4000
-LIBS:adc-dac
-LIBS:memory
-LIBS:xilinx
-LIBS:microcontrollers
-LIBS:dsp
-LIBS:microchip
-LIBS:analog_switches
-LIBS:motorola
-LIBS:texas
-LIBS:intel
-LIBS:audio
-LIBS:interface
-LIBS:digital-audio
-LIBS:philips
-LIBS:display
-LIBS:cypress
-LIBS:siliconi
-LIBS:opto
-LIBS:atmel
-LIBS:contrib
-LIBS:valves
-LIBS:PCIe_Mini_Adapter-cache
-EELAYER 25 0
+EESchema Schematic File Version 4
+EELAYER 26 0
 EELAYER END
 $Descr A4 11693 8268
@@
 $EndDescr
 $Comp
-L Conn_02x26_Odd_Even J1
+L Connector_Generic:Conn_02x26_Odd_Even J1
 U 1 1 5B8AACC8
 P 5800 2800
@@
 PIN48
 $Comp
-L Conn_01x15 J3
+L Connector_Generic:Conn_01x15 J3
 U 1 1 5B8ACE67
 P 8350 3400
@@
 PIN47
 $Comp
-L Conn_02x26_Counter_Clockwise J2
+L Connector_Generic:Conn_02x26_Counter_Clockwise J2
 U 1 1 5BAB0545
 P 7000 2800
